File: _autosave-rc2014-icecore.kicad_pcb (KiCad board)
At the start: 2 copper layers, 100 x 60.4 mm, 50 parts, among them J1 Conn_02x40_Top_Bottom, J2 Config, J3 DB15_Female_HighDensity_Mount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, P1 Mini-DIN_6pins_ver2, U1 SN74CB3T3245, U2 SN74CB3T3245, U3 SN74CB3T3245, U4 SN74CB3T3245, U5 SN74CB3T3245, U6 LM1117-3.3

Commit message: WIP
Parts:
- removed P1: Mini-DIN_6pins_ver2, 4x1md:Connector_Mini-DIN_Female_6Pin_2rows
- removed R1, R10, R11, R12, R16, R17, R18, R19, R2, R20, R24, R3, R4, R8, R9: 536, Resistor_SMD:R_0603_1608Metric
- removed R13, R14, R15, R21, R22, R23, R5, R6, R7: 270, Resistor_SMD:R_0603_1608Metric
- removed R25, R26: 100, Resistor_SMD:R_0603_1608Metric
- added J4: Conn_02x15_Odd_Even, Connector_PinSocket_2.54mm:PinSocket_2x15_P2.54mm_Horizontal, F.Cu at (177.0, 156.7)
- added J5: Conn_02x13_Odd_Even, Connector_PinHeader_2.54mm:PinHeader_2x13_P2.54mm_Horizontal, F.Cu at (65.3, 142.0)
- J3: value DB15_Female_HighDensity_MountingHoles -> Conn_02x15_Odd_Even; footprint Connector_Dsub:DSUB-15-HD_Female_Horizontal_P2.29x1.98mm_EdgePinOffset3.03mm_Housed_MountingHolesOffset4.94mm -> Connector_PinSocket_2.54mm:PinSocket_2x15_P2.54mm_Horizontal
- moved A1 58.3 mm to (124.7, 156.7), turned to 180 degrees
- moved J3 53.6 mm to (124.2, 91.9), turned to 270 degrees
- moved C11 24.7 mm to (127.1, 123.5)
- moved C7 24.7 mm to (123.3, 128.0)
- moved C6 24.7 mm to (127.3, 117.1)
- moved C12 24.7 mm to (131.4, 128.0)
Connections:
- A1 pad 1: /A14LV -> (no net)
- A1 pad 10: /CLKLV -> /P17
- A1 pad 100: (no net) -> /P55
- A1 pad 11: /MREQLV -> /P20
- A1 pad 12: //RDLV -> /P21
- A1 pad 13: /D0LV -> (no net)
- A1 pad 14: /D2LV -> (no net)
- A1 pad 15: /D4LV -> (no net)
- A1 pad 16: /D6LV -> (no net)
- A1 pad 17: /VGA_R0 -> /P32
- A1 pad 18: /VGA_R1 -> /P33
- A1 pad 19: /VGA_R2 -> /P36
- A1 pad 2: /A12LV -> (no net)
- A1 pad 20: /VGA_G0 -> /P37
- A1 pad 21: /VGA_G1 -> /P40
- A1 pad 22: /VGA_G2 -> /P41
- A1 pad 23: /VGA_B0 -> /P44
- A1 pad 24: /VGA_B1 -> /P45
- A1 pad 26: /A15LV -> (no net)
- A1 pad 27: /A13LV -> (no net)
- A1 pad 28: /A11LV -> (no net)
- A1 pad 29: /A9LV -> (no net)
- A1 pad 3: /A10LV -> (no net)
- A1 pad 30: /A7LV -> (no net)
- A1 pad 31: /A5LV -> (no net)
- A1 pad 32: /A3LV -> (no net)
- A1 pad 33: /A1LV -> (no net)
- A1 pad 34: //RESETLV -> /P18
- A1 pad 35: /INTLV -> /P19
- A1 pad 36: //WRLV -> /P22
- A1 pad 37: //IORQLV -> /P23
- A1 pad 38: /D1LV -> (no net)
- A1 pad 39: /D3LV -> (no net)
- A1 pad 4: /A8LV -> (no net)
- A1 pad 40: /D5LV -> (no net)
- A1 pad 41: /D7LV -> (no net)
- A1 pad 42: /VGA_HS -> /P34
- A1 pad 43: /VGA_VS -> /P35
- A1 pad 44: /VGA_B2 -> /P38
- A1 pad 45: (no net) -> /P39
- A1 pad 46: (no net) -> /P42
- A1 pad 47: (no net) -> /P43
- A1 pad 48: (no net) -> /P46
- A1 pad 49: (no net) -> /P47
- A1 pad 5: /A6LV -> (no net)
- A1 pad 50: (no net) -> /FPGA_VCC
- A1 pad 52: (no net) -> /SWDIO
- A1 pad 53: (no net) -> /SWCLK
- A1 pad 54: (no net) -> /~RESET
- A1 pad 6: /A4LV -> (no net)
- A1 pad 60: (no net) -> /AN5
- A1 pad 61: (no net) -> /AN6
- A1 pad 62: (no net) -> /AN7
- A1 pad 63: (no net) -> /AN8
- A1 pad 64: (no net) -> /AN9
- A1 pad 65: (no net) -> /AN11
- A1 pad 66: (no net) -> /AN13
- A1 pad 7: /A2LV -> (no net)
- A1 pad 76: (no net) -> GND
- A1 pad 77: (no net) -> /~ESS
- A1 pad 78: (no net) -> /TX
- A1 pad 79: (no net) -> /RX
- A1 pad 8: /A0LV -> (no net)
- A1 pad 80: (no net) -> /ESCK
- A1 pad 81: (no net) -> /EMISO
- A1 pad 82: (no net) -> /EMOSI
- A1 pad 83: (no net) -> /SCL
- A1 pad 84: (no net) -> /SDA
- A1 pad 85: (no net) -> /TMS
- A1 pad 86: (no net) -> /TDO
- A1 pad 87: (no net) -> /TDI
- A1 pad 88: (no net) -> /TCK
- A1 pad 89: (no net) -> +5V
- A1 pad 9: /M1LV -> /P16
- A1 pad 90: (no net) -> /AN10
- A1 pad 91: (no net) -> /AN12
- A1 pad 92: (no net) -> /AN14
- A1 pad 93: (no net) -> /P48
- A1 pad 94: (no net) -> /P49
- A1 pad 95: (no net) -> /P50
- A1 pad 96: (no net) -> /P51
- A1 pad 97: (no net) -> /P52
- A1 pad 98: (no net) -> /P53
- A1 pad 99: (no net) -> /P54
- J1 pad 69: (no net) -> /TX
- J1 pad 71: (no net) -> /RX
- J2 pad 11: /DATA_OE -> (no net)
- J2 pad 13: /SIG_OE -> (no net)
- J2 pad 15: /SIG2_OE -> (no net)
- J2 pad 9: /ADDR_OE -> (no net)
- J3 pad 1: Net-(J3-Pad1) -> +3V3
- J3 pad 10: GND -> /P36
- J3 pad 11: (no net) -> /P39
- J3 pad 12: (no net) -> /P37
- J3 pad 13: Net-(J3-Pad13) -> /AN9
- J3 pad 14: Net-(J3-Pad14) -> /AN8
- J3 pad 15: (no net) -> +5V
- J3 pad 2: Net-(J3-Pad2) -> +3V3
- J3 pad 3: Net-(J3-Pad3) -> GND
- J3 pad 4: (no net) -> GND
- J3 pad 5: GND -> /P34
- J3 pad 6: GND -> /P32
- J3 pad 7: GND -> /P35
- J3 pad 8: GND -> /P33
- J3 pad 9: (no net) -> /P38
- JP1 pad 3: (no net) -> /FPGA_VCC
- U1 pad 11: /A8LV -> (no net)
- U1 pad 12: /A9LV -> (no net)
- U1 pad 13: /A10LV -> (no net)
- U1 pad 14: /A11LV -> (no net)
- U1 pad 15: /A12LV -> (no net)
- U1 pad 16: /A13LV -> (no net)
- U1 pad 17: /A14LV -> (no net)
- U1 pad 18: /A15LV -> (no net)
- U1 pad 19: /ADDR_OE -> /RC_OE
- U2 pad 11: /A0LV -> (no net)
- U2 pad 12: /A1LV -> (no net)
- U2 pad 13: /A2LV -> (no net)
- U2 pad 14: /A3LV -> (no net)
- U2 pad 15: /A4LV -> (no net)
- U2 pad 16: /A5LV -> (no net)
- U2 pad 17: /A6LV -> (no net)
- U2 pad 18: /A7LV -> (no net)
- U2 pad 19: /ADDR_OE -> /RC_OE
- U3 pad 11: //IORQLV -> (no net)
- U3 pad 12: //RDLV -> (no net)
- U3 pad 13: //WRLV -> (no net)
- U3 pad 14: /MREQLV -> (no net)
- U3 pad 15: /M1LV -> (no net)
- U3 pad 19: /SIG_OE -> /RC_OE
- U4 pad 11: /INTLV -> (no net)
- U4 pad 12: /CLKLV -> (no net)
- U4 pad 13: //RESETLV -> (no net)
- U4 pad 19: /SIG2_OE -> /RC_OE
- U5 pad 11: /D7LV -> (no net)
- U5 pad 12: /D6LV -> (no net)
- U5 pad 13: /D5LV -> (no net)
- U5 pad 14: /D4LV -> (no net)
- U5 pad 15: /D3LV -> (no net)
- U5 pad 16: /D2LV -> (no net)
- U5 pad 17: /D1LV -> (no net)
- U5 pad 18: /D0LV -> (no net)
- U5 pad 19: /DATA_OE -> /RC_OE
Routing:
- net (no net): track 0.00 -> 58.7 mm
- net /A10LV: track 34.3 -> 0.09 mm
- net /A12LV: track 34.3 -> 0.29 mm
- net /A13LV: track 30.6 -> 0.00 mm
- net /A11LV: track 30.6 -> 0.00 mm
- net /A9LV: track 30.5 -> 0.00 mm
- net /A15LV: track 30.5 -> 14.5 mm
- net /A8LV: track 34.2 -> 32.9 mm
- net /A14LV: track 39.3 -> 38.6 mm
Other:
- board size 100 x 60.4 mm -> 100.1 x 70.1 mm
