File: rc2014-icecore.sch (KiCad schematic (older format))
At the start: 50 parts, among them J1 Conn_02x40_Top_Bottom, J2 Config, J3 DB15_Female_HighDensity_Mount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, P1 Mini-DIN_6pins_ver2, U1 SN74CB3T3245, U2 SN74CB3T3245, U3 SN74CB3T3245, U4 SN74CB3T3245, U5 SN74CB3T3245, U6 LM1117-3.3

Commit message: WIP
Parts:
- removed J3: DB15_Female_HighDensity_MountingHoles, Connector_Dsub:DSUB-15-HD_Female_Horizontal_P2.29x1.98mm_EdgePinOffset3.03mm_Housed_MountingHolesOffset4.94mm, symbol Connector:DB15_Female_HighDensity_MountingHoles
- removed P1: Mini-DIN_6pins_ver2, 4x1md:Connector_Mini-DIN_Female_6Pin_2rows, symbol 4x1md:Mini-DIN_6pins_ver2
- removed R1, R10, R11, R12, R16, R17, R18, R19, R2, R20, R24, R3, R4, R8, R9: 536, Resistor_SMD:R_0603_1608Metric, symbol Device:R
- removed R13, R14, R15, R21, R22, R23, R5, R6, R7: 270, Resistor_SMD:R_0603_1608Metric, symbol Device:R
- removed R25, R26: 100, Resistor_SMD:R_0603_1608Metric, symbol Device:R
- added J3, J4: Conn_02x15_Odd_Even, Connector_PinSocket_2.54mm:PinSocket_2x15_P2.54mm_Horizontal, symbol Connector_Generic:Conn_02x15_Odd_Even
- added J5: Conn_02x13_Odd_Even, Connector_PinHeader_2.54mm:PinHeader_2x13_P2.54mm_Horizontal, symbol Connector_Generic:Conn_02x13_Odd_Even
Connections:
- net labels added: +3V3, AN0, AN1, AN10, AN11, AN12, AN13, AN14, AN2, AN3, AN4, AN5, AN6, AN7, AN8, AN9, DONE, EMISO, EMOSI, ESCK, P0, P1, P10, P11, P12, P13, P14, P15, P16, P17, P18, P19, P2, P20, P21, P22, P23, P24, P25, P26, P27, P28, P29, P3, P30, P31, P32, P33, P34, P35, P36, P37, P38, P39, P4, P40, P41, P42, P43, P44, P45, P46, P47, P48, P49, P5, P50, P51, P52, P53, P54, P55, P6, P7, P8, P9, SCL, SDA, SWCLK, SWDIO, TCK, TDI, TDO, TMS, ~ESS, ~RESET
- net labels removed: KBD_CLK, KBD_DATA, MOUSE_CLK, MOUSE_DATA, VGA_B0, VGA_B1, VGA_B2, VGA_B3, VGA_G0, VGA_G1, VGA_G2, VGA_G3, VGA_HS, VGA_R0, VGA_R1, VGA_R2, VGA_R3, VGA_VS
- wire segments 335 -> 407
- no-connect marks 44 -> 30
Other:
- moved on the sheet: C10, C11, C12, C3, C4, C5, C6, C7, C8, C9

Commit message: Board routed
Parts:
- removed C10, C11, C12, C8, C9: C, Capacitor_SMD:C_0603_1608Metric, symbol Device:C
- removed J2: Config, Connector_PinHeader_2.54mm:PinHeader_2x08_P2.54mm_Vertical, symbol Connector_Generic:Conn_02x08_Odd_Even
- removed J4: Conn_02x15_Odd_Even, Connector_PinSocket_2.54mm:PinSocket_2x15_P2.54mm_Horizontal, symbol Connector_Generic:Conn_02x15_Odd_Even
Connections:
- net labels added: BUSACK, ~BUSREQ, ~HALT, ~NMI, ~RFSH, ~WAIT
- net labels removed: /IORQLV, /RDLV, /RESETLV, /WRLV, A0LV, A10LV, A11LV, A12LV, A13LV, A14LV, A15LV, A16, A17, A18, A19, A1LV, A20, A21, A22, A23, A2LV, A3LV, A4LV, A5LV, A6LV, A7LV, A8LV, A9LV, ADDR_OE, AN0, AN1, AN10, AN11, AN12, AN13, AN14, AN2, AN3, AN4, CLKLV, D0LV, D1LV, D2LV, D3LV, D4LV, D5LV, D6LV, D7LV, DATA_OE, DONE, INTLV, M1LV, MREQLV, SIG2_OE, SIG_OE
- wire segments 407 -> 308
- no-connect marks 30 -> 62
Other:
- moved on the sheet: U2, U3, U4, U5

Commit message: Board redesign
Parts:
- removed J1: Conn_02x40_Top_Bottom, Connector_PinHeader_2.54mm:PinHeader_2x39_P2.54mm_Vertical, symbol Connector_Generic:Conn_02x39_Odd_Even
- added J1: Conn_01x39, rc2014:PinHeader_1x39_P2.54mm_Vertical_NoSilk, symbol Connector_Generic:Conn_01x39
- added J2: Conn_01x10, rc2014:PinHeader_1x10_P2.54mm_Vertical_NoSilk, symbol Connector_Generic:Conn_01x10
- added R1: R, symbol Device:R
- renumbered C7 to C3, C3 to C4, C4 to C5, C5 to C6, C6 to C7, J5 to J4, U6 to U1, U1 to U2, U2 to U3, U3 to U4, U4 to U5, U5 to U6
Connections:
- wire segments 308 -> 309
- no-connect marks 62 -> 28
Other:
- moved on the sheet: A1A, A1B, C1, C2, C3, C4, C5, C6, C7, J3, J4, JP1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

Commit message: 2nd redesign
Parts:
- added H1: MountingHole, MountingHole:MountingHole_3.2mm_M3, symbol Mechanical:MountingHole
- R1: footprint (none) -> Resistor_SMD:R_0603_1608Metric
Changed lines of the file:
@@
 F 0 "R1" V 5033 890 50  0000 C CNN
 F 1 "R" V 5124 890 50  0000 C CNN
-F 2 "" V 5170 890 50  0001 C CNN
+F 2 "Resistor_SMD:R_0603_1608Metric" V 5170 890 50  0001 C CNN
 F 3 "~" H 5240 890 50  0001 C CNN
 	1    5240 890
@@
 Wire Wire Line
 	5390 890  5460 890
+$Comp
+L Mechanical:MountingHole H1
+U 1 1 66CA3A6A
+P 860 6610
+F 0 "H1" H 960 6656 50  0000 L CNN
+F 1 "MountingHole" H 960 6565 50  0000 L CNN
+F 2 "MountingHole:MountingHole_3.2mm_M3" H 860 6610 50  0001 C CNN
+F 3 "~" H 860 6610 50  0001 C CNN
+	1    860  6610
+	1    0    0    -1
+$EndComp
 $EndSCHEMATC

Commit message: reorder pmod pins
Changed lines of the file:
@@
 Text Label 8380 6260 0    50   ~ 0
 P42
-Text Label 9230 6260 0    50   ~ 0
+Text Label 8380 6160 0    50   ~ 0
 P43
 Text Label 9230 6060 0    50   ~ 0
@@
 Text Label 9230 5960 0    50   ~ 0
 P45
-Text Label 8380 6160 0    50   ~ 0
+Text Label 9230 6260 0    50   ~ 0
 P46
 Text Label 9230 6160 0    50   ~ 0

Commit message: WIP
Parts:
- removed C1: 100nF, Capacitor_SMD:C_0603_1608Metric, symbol Device:CP_Small
- removed C2: 10uF, Capacitor_SMD:C_0603_1608Metric, symbol Device:CP_Small
- removed C3, C4, C5, C6, C7: C, Capacitor_SMD:C_0603_1608Metric, symbol Device:C
- removed H1: MountingHole, MountingHole:MountingHole_3.2mm_M3, symbol Mechanical:MountingHole
- removed J1: Conn_01x39, rc2014:PinHeader_1x39_P2.54mm_Vertical_NoSilk, symbol Connector_Generic:Conn_01x39
- removed J2: Conn_01x10, rc2014:PinHeader_1x10_P2.54mm_Vertical_NoSilk, symbol Connector_Generic:Conn_01x10
- removed JP1: Ext Power, Connector_PinHeader_2.54mm:PinHeader_1x03_P2.54mm_Vertical, symbol Jumper:Jumper_3_Bridged12
- removed R1: R, Resistor_SMD:R_0603_1608Metric, symbol Device:R
- removed U1: LM1117-3.3, Package_TO_SOT_SMD:SOT-223-3_TabPin2, symbol rc2014-icecore-rescue:LM1117-3.3
- removed U2, U3, U4, U5, U6: SN74CB3T3245, Package_SO:TSSOP-20_4.4x6.5mm_P0.65mm, symbol rc2014-icecore:SN74CB3T3245
- added J1: Conn_02x25_Odd_Even, Connector_PinHeader_2.54mm:PinHeader_2x25_P2.54mm_Vertical, symbol Connector_Generic:Conn_02x25_Odd_Even
- J2: renamed from J3; footprint Connector_PinSocket_2.54mm:PinSocket_2x15_P2.54mm_Horizontal -> Connector_PinSocket_2.54mm:PinSocket_2x15_P2.54mm_Vertical
- J3: renamed from J4; footprint Connector_PinHeader_2.54mm:PinHeader_2x13_P2.54mm_Horizontal -> Connector_PinHeader_2.54mm:PinHeader_2x13_P2.54mm_Vertical
Connections:
- net labels removed: +3.3V, +3V3, /IORQ, /RD, /RESET, /WR, 5V, A0, A1, A10, A11, A12, A13, A14, A15, A2, A3, A4, A5, A6, A7, A8, A9, BUSACK, CLK, D0, D1, D2, D3, D4, D5, D6, D7, INT, M1, MREQ, RC_OE, ~BUSREQ, ~HALT, ~NMI, ~RFSH, ~WAIT
- wire segments 309 -> 209
- no-connect marks 28 -> 27
