File: rc2014-icecore.sch (KiCad schematic (older format))
At the start: 4 parts, among them J1 Conn_02x25_Odd_Even, J2 Conn_02x15_Odd_Even, J3 Conn_02x13_Odd_Even

Commit message: Start new merged design
Parts:
- added C1: 100nF, Capacitor_SMD:C_0603_1608Metric, symbol Device:CP_Small
- added C2: 10uF, Capacitor_SMD:C_0603_1608Metric, symbol Device:CP_Small
- added C3, C4, C5, C6, C7: C, Capacitor_SMD:C_0603_1608Metric, symbol Device:C
- added J1: Conn_01x39, rc2014:PinHeader_1x39_P2.54mm_Vertical_NoSilk, symbol Connector_Generic:Conn_01x39
- added J2: Conn_01x10, rc2014:PinHeader_1x10_P2.54mm_Vertical_NoSilk, symbol Connector_Generic:Conn_01x10
- added J3: Conn_02x25_Odd_Even, Connector_PinSocket_2.54mm:PinSocket_2x25_P2.54mm_Vertical, symbol Connector_Generic:Conn_02x25_Odd_Even
- added JP1: Ext Power, Connector_PinHeader_2.54mm:PinHeader_1x03_P2.54mm_Vertical, symbol Jumper:Jumper_3_Bridged12
- added JP2: Jumper, Connector_PinHeader_2.54mm:PinHeader_1x02_P2.54mm_Vertical, symbol Device:Jumper
- added R1: R, Resistor_SMD:R_0603_1608Metric, symbol Device:R
- added U1: LM1117-3.3, Package_TO_SOT_SMD:SOT-223-3_TabPin2, symbol rc2014-icecore-rescue:LM1117-3.3
- added U2, U3, U4, U5, U6: SN74CB3T3245, Package_SO:TSSOP-20_4.4x6.5mm_P0.65mm, symbol rc2014-icecore:SN74CB3T3245
Connections:
- net labels added: +3.3V, /IORQ, /RD, /RESET, /WR, 5V, A0, A1, A10, A11, A12, A13, A14, A15, A2, A3, A4, A5, A6, A7, A8, A9, BUSACK, CLK, D0, D1, D2, D3, D4, D5, D6, D7, INT, M1, MREQ, RC_OE, ~BUSREQ, ~HALT, ~NMI, ~RFSH, ~WAIT
- wire segments 209 -> 416
- no-connect marks 27 -> 39
Other:
- moved on the sheet: A1A, A1B, J1, J2, J3

Commit message: Further work on combining boards - still WIP
Parts:
- removed J1: Conn_02x25_Odd_Even, Connector_PinHeader_2.54mm:PinHeader_2x25_P2.54mm_Vertical, symbol Connector_Generic:Conn_02x25_Odd_Even
- removed J1: Conn_01x39, rc2014:PinHeader_1x39_P2.54mm_Vertical_NoSilk, symbol Connector_Generic:Conn_01x39
- removed J2: Conn_01x10, rc2014:PinHeader_1x10_P2.54mm_Vertical_NoSilk, symbol Connector_Generic:Conn_01x10
- removed J3: Conn_02x25_Odd_Even, Connector_PinSocket_2.54mm:PinSocket_2x25_P2.54mm_Vertical, symbol Connector_Generic:Conn_02x25_Odd_Even
- added J1: Conn_02x40_Top_Bottom, Connector_PinHeader_2.54mm:PinHeader_2x40_P2.54mm_Vertical, symbol Connector_Generic:Conn_02x40_Top_Bottom
- added J2: Conn_02x04_Counter_Clockwise, Connector_PinHeader_2.54mm:PinHeader_1x06_P2.54mm_Vertical, symbol Connector_Generic:Conn_01x06
- added JP3, JP4, JP5: SolderJumper_2_Bridged, Jumper:SolderJumper-2_P1.3mm_Bridged_RoundedPad1.0x1.5mm, symbol Jumper:SolderJumper_2_Bridged
- renumbered J2 to J3, J3 to J4, U5 to U1, U6 to U2, U4 to U3, U2 to U4, U3 to U5, U1 to U6
Connections:
- net labels added: LVX1, X1, X2
- wire segments 416 -> 326
- no-connect marks 39 -> 61
Other:
- moved on the sheet: A1B, JP2, R1, U1, U2, U3, U4, U5
