File: rc2014-icecore.kicad_pcb (KiCad board)
At the start: 2 copper layers, 99.3 x 96.8 mm, 27 parts, among them J1 Conn_01x39, J1 Conn_02x25_Odd_Even, J2 Conn_01x10, J2 Conn_02x15_Odd_Even, J3 Conn_02x13_Odd_Even, J3 Conn_02x25_Odd_Even, U1 LM1117-3.3, U2 SN74CB3T3245, U3 SN74CB3T3245, U4 SN74CB3T3245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

Commit message: Further work on combining boards - still WIP
Parts:
- removed G***: LOGO, rc2014:blackedge
- removed G***: LOGO, rc2014:maxreal
- removed the J1 at (61.7, 163.3)
- removed the J1 at (69.0, 124.6)
- removed the J2 at (102.4, 160.8)
- removed the J2 at (130.3, 112.2)
- removed the J3 at (65.5, 143.6)
- removed the J3 at (68.1, 117.3)
- removed the REF** at (119.8, 104.9)
- added J1: Conn_02x40_Top_Bottom, Connector_PinHeader_2.54mm:PinHeader_2x40_P2.54mm_Vertical, F.Cu at (61.7, 163.3)
- added J2: Conn_02x04_Counter_Clockwise, Connector_PinHeader_2.54mm:PinHeader_1x06_P2.54mm_Vertical, F.Cu at (128.3, 156.2)
- added J3: Conn_02x15_Odd_Even, Connector_PinSocket_2.54mm:PinSocket_2x15_P2.54mm_Vertical, F.Cu at (62.5, 154.9)
- added J4: Conn_02x13_Odd_Even, Connector_PinHeader_2.54mm:PinHeader_2x13_P2.54mm_Vertical, F.Cu at (126.7, 108.7)
- added JP3: SolderJumper_2_Bridged, Jumper:SolderJumper-2_P1.3mm_Bridged_RoundedPad1.0x1.5mm, F.Cu at (102.3, 46.0)
- added JP4: SolderJumper_2_Bridged, Jumper:SolderJumper-2_P1.3mm_Bridged_RoundedPad1.0x1.5mm, F.Cu at (106.7, 46.0)
- added JP5: SolderJumper_2_Bridged, Jumper:SolderJumper-2_P1.3mm_Bridged_RoundedPad1.0x1.5mm, F.Cu at (111.0, 46.0)
- U1: value LM1117-3.3 -> SN74CB3T3245; footprint Package_TO_SOT_SMD:SOT-223-3_TabPin2 -> Package_SO:TSSOP-20_4.4x6.5mm_P0.65mm
- U6: value SN74CB3T3245 -> LM1117-3.3; footprint Package_SO:TSSOP-20_4.4x6.5mm_P0.65mm -> Package_TO_SOT_SMD:SOT-223-3_TabPin2
- moved C3 126.0 mm to (242.1, 91.7)
- moved C4 126.0 mm to (176.1, 91.7)
- moved C5 126.0 mm to (192.4, 91.7)
- moved C7 126.0 mm to (225.7, 91.7)
- moved R1 126.0 mm to (176.0, 96.0)
- moved U2 126.0 mm to (181.0, 93.7)
- moved U3 126.0 mm to (197.2, 93.7)
- moved C6 126.0 mm to (208.9, 91.7)
- moved U4 98.2 mm to (190.2, 109.0)
- moved U5 90.7 mm to (199.4, 110.5)
- moved U1 72.1 mm to (209.8, 111.3)
- moved A1 38.4 mm to (82.0, 107.4)
Connections:
- A1 pad 89: +5V -> Net-(A1-Pad89)
- JP2 pad 1: Net-(J3-Pad45) -> Net-(A1-Pad89)
- U1 pad 1: GND -> (no net)
- U1 pad 2: Net-(C2-Pad1) -> /MREQ
- U1 pad 3: +5V -> /~HALT
- U2 pad 11: /P7 -> /P55
- U2 pad 12: /P6 -> /P54
- U2 pad 13: /P5 -> /P53
- U2 pad 14: /P4 -> /P52
- U2 pad 15: /P3 -> /P51
- U2 pad 16: /P2 -> /P50
- U2 pad 17: /P1 -> /P49
- U2 pad 18: /P0 -> /P48
- U2 pad 2: /A15 -> /D0
- U2 pad 3: /A14 -> /D1
- U2 pad 4: /A13 -> /D2
- U2 pad 5: /A12 -> /D3
- U2 pad 6: /A11 -> /D4
- U2 pad 7: /A10 -> /D5
- U2 pad 8: /A9 -> /D6
- U2 pad 9: /A8 -> /D7
- U3 pad 11: /P15 -> /P22
- U3 pad 12: /P14 -> /P21
- U3 pad 13: /P13 -> /P20
- U3 pad 14: /P12 -> /P19
- U3 pad 15: /P11 -> /P18
- U3 pad 16: /P10 -> /P17
- U3 pad 17: /P9 -> /P16
- U3 pad 18: /P8 -> /LVX1
- U3 pad 2: /A7 -> /X1
- U3 pad 3: /A6 -> /X2
- U3 pad 4: /A5 -> /M1
- U3 pad 5: /A4 -> /~RFSH
- U3 pad 6: /A3 -> //RESET
- U3 pad 7: /A2 -> /CLK
- U3 pad 8: /A1 -> /INT
- U3 pad 9: /A0 -> /BUSACK
- U4 pad 11: /P22 -> /P7
- U4 pad 12: /P21 -> /P6
- U4 pad 13: /P20 -> /P5
- U4 pad 14: /P19 -> /P4
- U4 pad 15: /P18 -> /P3
- U4 pad 16: /P17 -> /P2
- U4 pad 17: GND -> /P1
- U4 pad 18: GND -> /P0
- U4 pad 2: GND -> /A15
- U4 pad 3: GND -> /A14
- U4 pad 4: /M1 -> /A13
- U4 pad 5: /~RFSH -> /A12
- U4 pad 6: //RESET -> /A11
- U4 pad 7: /CLK -> /A10
- U4 pad 8: /INT -> /A9
- U4 pad 9: /BUSACK -> /A8
- U5 pad 11: /P31 -> /P15
- U5 pad 12: /P30 -> /P14
- U5 pad 13: /P29 -> /P13
- U5 pad 14: /P28 -> /P12
- U5 pad 15: /P27 -> /P11
- U5 pad 16: /P26 -> /P10
- U5 pad 17: /P25 -> /P9
- U5 pad 18: /P24 -> /P8
- U5 pad 2: /MREQ -> /A7
- U5 pad 3: /~HALT -> /A6
- U5 pad 4: //WR -> /A5
- U5 pad 5: /~BUSREQ -> /A4
- U5 pad 6: //RD -> /A3
- U5 pad 7: /~WAIT -> /A2
- U5 pad 8: //IORQ -> /A1
- U5 pad 9: /~NMI -> /A0
- U6 pad 1: (no net) -> GND
- U6 pad 2: /D0 -> Net-(C2-Pad1)
- U6 pad 3: /D1 -> +5V
Routing:
- net GND: track 237.4 -> 0.00 mm, vias 17 -> 0
- net /P23: track 148.9 -> 0.00 mm, vias 1 -> 0
- net /P24: track 124.3 -> 0.00 mm
- net +5V: track 118.9 -> 0.00 mm, vias 1 -> 0
- net /FPGA_VCC: track 104.0 -> 0.00 mm, vias 3 -> 0
- net /P9: track 103.6 -> 0.00 mm
- net +3V3: track 100.5 -> 0.00 mm
- net /P17: track 89.1 -> 0.00 mm, vias 1 -> 0
- net /P25: track 83.9 -> 0.00 mm, vias 1 -> 0
- net /P27: track 81.4 -> 0.00 mm, vias 2 -> 0
- net /P26: track 80.7 -> 0.00 mm, vias 1 -> 0
- net /P28: track 80.5 -> 0.00 mm, vias 1 -> 0
- net /P20: track 80.3 -> 0.00 mm, vias 1 -> 0
- net /P29: track 79.9 -> 0.00 mm, vias 1 -> 0
- net /P8: track 78.8 -> 0.00 mm
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Other:
- board size 99.3 x 96.8 mm -> 99.6 x 62 mm

Commit message: partially routed
Parts:
- removed JP3, JP4, JP5: SolderJumper_2_Bridged, Jumper:SolderJumper-2_P1.3mm_Bridged_RoundedPad1.0x1.5mm
- removed the U1 at (209.8, 111.3)
- added U2: SN74CB3T3245, Package_SO:TSSOP-20_4.4x6.5mm_P0.65mm, F.Cu at (117.2, 127.5)
- J1: value Conn_02x40_Top_Bottom -> Conn_01x39; footprint Connector_PinHeader_2.54mm:PinHeader_2x40_P2.54mm_Vertical -> rc2014:PinHeader_1x39_P2.54mm_Vertical_NoSilk
- J2: value Conn_02x04_Counter_Clockwise -> Conn_01x10; footprint Connector_PinHeader_2.54mm:PinHeader_1x06_P2.54mm_Vertical -> rc2014:PinHeader_1x10_P2.54mm_Vertical_NoSilk
- moved C3 134.0 mm to (112.4, 125.4)
- moved C7 130.8 mm to (102.6, 135.9)
- moved C6 119.6 mm to (94.2, 125.4)
- moved C5 116.4 mm to (84.8, 136.0)
- moved U5 116.4 mm to (89.6, 138.0)
- moved R1 104.8 mm to (76.9, 129.9)
- moved C4 104.8 mm to (77.0, 125.6)
- moved U4 104.8 mm to (81.9, 127.7)
- moved U1 96.0 mm to (107.4, 137.9)
- moved U3 93.1 mm to (99.0, 127.4)
- moved J4 77.9 mm to (65.0, 156.2), turned to 180 degrees
- moved J3 64.9 mm to (127.0, 147.8)
- moved J2 26.3 mm to (102.4, 160.8), turned to 90 degrees
- moved C1 19.5 mm to (128.1, 153.3)
- moved C2 19.5 mm to (137.3, 153.3)
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- renumbered JP2 to JP1, JP1 to JP2, U5 to U1, U4 to U3, U2 to U4, U3 to U5
Connections:
- A1 pad 89: Net-(A1-Pad89) -> +5V
- A1 pad 9: /P16 -> (no net)
- J2 pad 2: /LVX1 -> +5V
- J2 pad 3: /X1 -> /~RFSH
- J2 pad 4: /X2 -> (no net)
- J2 pad 5: +3V3 -> (no net)
- J2 pad 6: +5V -> /BUSACK
- JP1 pad 1: Net-(A1-Pad89) -> (no net)
- U1 pad 11: /P15 -> /P31
- U1 pad 12: /P14 -> /P30
- U1 pad 13: /P13 -> /P29
- U1 pad 14: /P12 -> /P28
- U1 pad 15: /P11 -> /P27
- U1 pad 16: /P10 -> /P26
- U1 pad 17: /P9 -> /P25
- U1 pad 18: /P8 -> /P24
- U1 pad 2: /A7 -> /MREQ
- U1 pad 3: /A6 -> /~HALT
- U1 pad 4: /A5 -> //WR
- U1 pad 5: /A4 -> /~BUSREQ
- U1 pad 6: /A3 -> //RD
- U1 pad 7: /A2 -> /~WAIT
- U1 pad 8: /A1 -> //IORQ
- U1 pad 9: /A0 -> /~NMI
- U3 pad 11: /P7 -> /P22
- U3 pad 12: /P6 -> /P21
- U3 pad 13: /P5 -> /P20
- U3 pad 14: /P4 -> /P19
- U3 pad 15: /P3 -> /P18
- U3 pad 16: /P2 -> /P17
- U3 pad 17: /P1 -> GND
- U3 pad 18: /P0 -> GND
- U3 pad 2: /A15 -> GND
- U3 pad 3: /A14 -> GND
- U3 pad 4: /A13 -> /M1
- U3 pad 5: /A12 -> /~RFSH
- U3 pad 6: /A11 -> //RESET
- U3 pad 7: /A10 -> /CLK
- U3 pad 8: /A9 -> /INT
- U3 pad 9: /A8 -> /BUSACK
- U4 pad 11: /P55 -> /P7
- U4 pad 12: /P54 -> /P6
- U4 pad 13: /P53 -> /P5
- U4 pad 14: /P52 -> /P4
- U4 pad 15: /P51 -> /P3
- U4 pad 16: /P50 -> /P2
- U4 pad 17: /P49 -> /P1
- U4 pad 18: /P48 -> /P0
- U4 pad 2: /D0 -> /A15
- U4 pad 3: /D1 -> /A14
- U4 pad 4: /D2 -> /A13
- U4 pad 5: /D3 -> /A12
- U4 pad 6: /D4 -> /A11
- U4 pad 7: /D5 -> /A10
- U4 pad 8: /D6 -> /A9
- U4 pad 9: /D7 -> /A8
- U5 pad 11: /P22 -> /P15
- U5 pad 12: /P21 -> /P14
- U5 pad 13: /P20 -> /P13
- U5 pad 14: /P19 -> /P12
- U5 pad 15: /P18 -> /P11
- U5 pad 16: /P17 -> /P10
- U5 pad 17: /P16 -> /P9
- U5 pad 18: /LVX1 -> /P8
- U5 pad 2: /X1 -> /A7
- U5 pad 3: /X2 -> /A6
- U5 pad 4: /M1 -> /A5
- U5 pad 5: /~RFSH -> /A4
- U5 pad 6: //RESET -> /A3
- U5 pad 7: /CLK -> /A2
- U5 pad 8: /INT -> /A1
- U5 pad 9: /BUSACK -> /A0
Routing:
- net /D7: track 0.00 -> 49.3 mm
- net /D6: track 0.00 -> 48.4 mm
- net /D5: track 0.00 -> 46.6 mm
- net /D4: track 0.00 -> 44.7 mm
- net /D3: track 0.00 -> 42.8 mm
- net /D2: track 0.00 -> 40.9 mm
- net /CLK: track 0.00 -> 40.4 mm
- net /A15: track 0.00 -> 40.2 mm
- net //RESET: track 0.00 -> 39.6 mm
- net /INT: track 0.00 -> 39.6 mm
- net /A14: track 0.00 -> 39.4 mm
- net /M1: track 0.00 -> 39.4 mm
- net /D1: track 0.00 -> 39.1 mm
- net /A13: track 0.00 -> 38.6 mm
- net /D0: track 0.00 -> 38.3 mm
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Other:
- board size 99.6 x 62 mm -> 99.3 x 57.2 mm
